Commit message: add ros2_control differential controller for Gazebo

File: rb1_ros2_description/urdf/common.gazebo.xacro (robot description, xacro)
@@ -2,6 +2,38 @@
 <robot xmlns:xacro="http://www.ros.org/wiki/xacro">
 	<!-- ROS CONTROL GAZEBO PLUGIN -->
-    <!-- <xacro:macro name="ros2_control">
-	</xacro:macro> -->
+    <xacro:macro name="rb1_diff_drive_system" params="prefix robot_name">
+    <ros2_control name="Rb1DiffDriveSystem" type="system">
+      <hardware>
+          <plugin>gazebo_ros2_control/GazeboSystem</plugin>
+      </hardware>
+      <joint name="${prefix}left_wheel_joint">
+        <command_interface name="velocity">
+          <param name="min">-100</param>
+          <param name="max">100</param>
+        </command_interface>
+        <state_interface name="position"/>
+        <state_interface name="velocity"/>
+        <state_interface name="effort"/>
+      </joint>
+      <joint name="${prefix}right_wheel_joint">
+        <command_interface name="velocity">
+          <param name="min">-100</param>
+          <param name="max">100</param>
+        </command_interface>
+        <state_interface name="position"/>
+        <state_interface name="velocity"/>
+        <state_interface name="effort"/>
+      </joint>
+    </ros2_control>
+    <gazebo>
+      <plugin filename="libgazebo_ros2_control.so" name="gazebo_ros2_control">
+        <ros>
+          <namespace>/${robot_name}</namespace>
+          <!--<remapping>~/out:=joint_states</remapping>-->
+        </ros>
+        <parameters>$(find rb1_ros2_description)/config/rb1_controller.yaml</parameters>
+      </plugin>
+    </gazebo>
+	</xacro:macro>
 	<xacro:macro name="gazebo_colors" params="prefix">
 		<gazebo reference="$(arg prefix)base_footprint">

File: rb1_ros2_description/xacro/rb1_ros2_base.urdf.xacro (robot description, xacro)
@@ -41,4 +41,5 @@
 	<xacro:property name="elevator_z" value="0.213" />
 	<xacro:arg name="prefix" default="robot_"/>
+    <xacro:arg name="robot_name" default="robot_"/>
 	<xacro:arg name="ros_planar_move_plugin" default="false"/>
 	<xacro:arg name="gpu" default="false"/>
@@ -85,4 +86,4 @@
 	</xacro:sensor_orbbec_astra>
 	<!-- Gazebo ros2 control plugins -->
-	<!-- <xacro:ros2_control/> -->
+	<xacro:rb1_diff_drive_system prefix="$(arg prefix)" robot_name="$(arg robot_name)"/>
 </robot>

Commit message: add elevator controller

File: rb1_ros2_description/urdf/common.gazebo.xacro (robot description, xacro)
@@ -25,4 +25,13 @@
         <state_interface name="effort"/>
       </joint>
+      <joint name="${prefix}elevator_platform_joint">
+        <command_interface name="position">
+          <param name="min">0.0</param>
+          <param name="max">0.034</param>
+        </command_interface>
+        <state_interface name="position"/>
+        <state_interface name="velocity"/>
+        <state_interface name="acceleration"/>
+      </joint>
     </ros2_control>
     <gazebo>
